File: design/balancebot.kicad_pcb (KiCad board)
At the start: 2 copper layers, 66.7 x 59.7 mm, 21 parts, among them J1 Switch, J2 11.1V Batt, J3 Passthrough, J4 Servo Interface, J5 Left Motor Interface, J6 Right Motor Interface, U1 ESP32, U2 L7805CV, U3 GY-521

Commit message: WIP PCB design update
Parts:
- removed the C1 at (-38.1, 6.60)
- removed the C2 at (-38.1, 4.06)
- removed the J6 at (-10.2, 31.1)
- removed REF** (x2): MountingHole_2.1mm, MountingHole:MountingHole_2.1mm
- added J3: Passthrough, balancebot-footprints:bb_PinSocket_1x19_P2.54mm_Vertical, F.Cu at (-59.8, -34.9)
- added TB1: Switch, balancebot-footprints:bb_TE_282837-2, F.Cu at (-40.0, 14.0)
- added TB2: 6.5V-36V, balancebot-footprints:bb_TE_282837-2, F.Cu at (-40.0, 24.1)
- J1: value Switch -> VIN Passthrough; footprint balancebot-footprints:bb_TE_282837-2 -> Connector_PinHeader_2.54mm:PinHeader_1x02_P2.54mm_Vertical
- J2: value 11.1V Batt -> 5V Passthrough; footprint balancebot-footprints:bb_TE_282837-2 -> Connector_PinHeader_2.54mm:PinHeader_1x02_P2.54mm_Vertical
- J4: renamed from J3; value Passthrough -> Servo Interface; footprint balancebot-footprints:bb_PinSocket_1x19_P2.54mm_Vertical -> Connector_PinHeader_2.54mm:PinHeader_1x03_P2.54mm_Vertical
- J5: renamed from J4; value Servo Interface -> Left Motor Interface; footprint Connector_PinHeader_2.54mm:PinHeader_1x03_P2.54mm_Vertical -> Connector_PinHeader_2.54mm:PinHeader_1x04_P2.54mm_Vertical
- J6: renamed from J5; value Left Motor Interface -> Right Motor Interface
- U2: value L7805CV -> TSR_1-2450; footprint Package_TO_SOT_THT:TO-220-3_Horizontal_TabDown -> Converter_DCDC:Converter_DCDC_TRACO_TSR-1_THT
- moved J5 55.9 mm to (-36.6, 63.6)
- moved J4 48.6 mm to (-77.9, -7.87)
- moved J2 45.8 mm to (-79.2, 1.59), turned to 0 degrees
- moved C1 44.5 mm to (-63.4, 18.8)
- moved J6 44.5 mm to (-69.7, 39.8)
- moved A1 44.5 mm to (-65.9, 26.4)
- moved U2 43.3 mm to (-72.1, -28.4), turned to 90 degrees
- moved C2 41.9 mm to (-30.2, 42.7)
- moved A2 41.9 mm to (-32.8, 50.3)
- moved J1 38.3 mm to (-75.6, 1.59), turned to 0 degrees
- moved U1 33.6 mm to (-10.4, -45.0)
- moved U3 32.2 mm to (44.5, 22.1)
- renumbered C3 to C1, C4 to C2
Connections:
- A1 pad 1: STEP_ENABLE -> MOTOR_ENABLE
- A1 pad 7: STEP_STEP_L -> LEFT_MOTOR_STEP
- A1 pad 8: STEP_DIR_L -> LEFT_MOTOR_DIR
- A2 pad 1: STEP_ENABLE -> MOTOR_ENABLE
- A2 pad 7: STEP_STEP_R -> RIGHT_MOTOR_STEP
- A2 pad 8: STEP_DIR_R -> RIGHT_MOTOR_DIR
- J1 pad 1: +BATT -> +VMOT
- J1 pad 2: +VMOT -> GND
- J2 pad 1: +BATT -> +5V
- J4 pad 1: +5V -> ARM_SERVO_PWM
- J4 pad 2: IO11 -> +5V
- J4 pad 3: IO10 -> GND
- J5 pad 1: SERVO_PWM -> Net-(A1-Pad14)
- J5 pad 2: +5V -> Net-(A1-Pad13)
- J5 pad 3: GND -> Net-(A1-Pad12)
- J6 pad 1: Net-(A1-Pad14) -> Net-(A2-Pad14)
- J6 pad 2: Net-(A1-Pad13) -> Net-(A2-Pad13)
- J6 pad 3: Net-(A1-Pad12) -> Net-(A2-Pad12)
- J6 pad 4: Net-(A1-Pad11) -> Net-(A2-Pad11)
- U1 pad 10: STEP_DIR_R -> RIGHT_MOTOR_DIR
- U1 pad 11: STEP_STEP_R -> RIGHT_MOTOR_STEP
- U1 pad 12: STEP_DIR_L -> LEFT_MOTOR_DIR
- U1 pad 13: STEP_STEP_L -> LEFT_MOTOR_STEP
- U1 pad 5: SERVO_PWM -> ARM_SERVO_PWM
- U1 pad 9: STEP_ENABLE -> MOTOR_ENABLE
Routing:
- net +5V: track 137.1 -> 0.00 mm
- net +3V3: track 88.8 -> 0.00 mm
- net +VMOT: track 74.6 -> 0.00 mm
- net MPU_SCL: track 69.8 -> 0.00 mm
- net MPU_SDA: track 69.3 -> 0.00 mm
- net MPU_INTERRUPT: track 66.4 -> 0.00 mm
- net STEP_DIR_L: track 40.3 -> 0.00 mm, vias 2 -> 0
- net STEP_STEP_L: track 37.4 -> 0.00 mm, vias 2 -> 0
- net STEP_ENABLE: track 35.5 -> 0.00 mm, vias 1 -> 0
- net SERVO_PWM: track 33.4 -> 0.00 mm
- net STEP_DIR_R: track 30.6 -> 0.00 mm, vias 2 -> 0
- net STEP_STEP_R: track 26.5 -> 0.00 mm, vias 2 -> 0
- net Net-(A1-Pad14): track 20.3 -> 0.00 mm
- net Net-(A2-Pad14): track 20.2 -> 0.00 mm
- net Net-(A2-Pad13): track 16.5 -> 0.00 mm
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Other:
- board text added: "BalanceBot by FrostieBot v0.3.4"
- board text added: "VIN"
- board text removed: "BalanceBot by FrostieBot v0.2.4"

Commit message: update PCB design to revision 0.4.5
Parts:
- removed J1: VIN Passthrough, Connector_PinHeader_2.54mm:PinHeader_1x02_P2.54mm_Vertical
- removed J2: 5V Passthrough, Connector_PinHeader_2.54mm:PinHeader_1x02_P2.54mm_Vertical
- TB2: value 6.5V-36V -> 8V-36V
- U2: value TSR_1-2450 -> OKI-78SR-5/1.5-W36-C; footprint Converter_DCDC:Converter_DCDC_TRACO_TSR-1_THT -> Converter_DCDC:Converter_DCDC_muRata_OKI-78SR_Vertical
- U3: value GY-521 -> MPU6050
- moved J4 261.5 mm to (157.4, 106.0)
- moved U2 260.8 mm to (159.4, 91.7), turned to 0 degrees
- moved J6 222.1 mm to (142.2, 106.0)
- moved J3 206.9 mm to (114.0, 77.3), turned to 90 degrees
- moved A1 205.2 mm to (128.7, 91.7)
- moved C1 205.2 mm to (131.2, 84.1)
- moved H4 195.5 mm to (167.3, 105.4)
- moved A2 183.5 mm to (146.1, 91.7)
- moved C2 183.5 mm to (148.6, 84.1)
- moved U1 182.7 mm to (136.9, 63.2)
- moved TB1 169.9 mm to (114.4, 84.7)
- moved TB2 169.9 mm to (114.4, 94.9)
- moved H1 169.8 mm to (110.0, 53.0)
- moved H2 168.8 mm to (110.0, 105.4)
- moved J5 166.9 mm to (124.8, 106.0)
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Connections:
- J3 pad 10: RIGHT_MOTOR_DIR -> RIGHT_MOTOR_STEP
- J3 pad 11: RIGHT_MOTOR_STEP -> MOTOR_ENABLE
- J3 pad 9: MOTOR_ENABLE -> RIGHT_MOTOR_DIR
- U1 pad 10: RIGHT_MOTOR_DIR -> RIGHT_MOTOR_STEP
- U1 pad 11: RIGHT_MOTOR_STEP -> MOTOR_ENABLE
- U1 pad 9: MOTOR_ENABLE -> RIGHT_MOTOR_DIR
Routing:
- net +3V3: track 0.00 -> 133.8 mm, vias 0 -> 1
- net +VMOT: track 0.00 -> 69.3 mm
- net +5V: track 0.00 -> 35.4 mm
- net ARM_SERVO_PWM: track 0.00 -> 34.7 mm
- net MOTOR_ENABLE: track 0.00 -> 33.5 mm
- net MPU_SCL: track 0.00 -> 33.0 mm, vias 0 -> 1
- net LEFT_MOTOR_DIR: track 0.00 -> 32.0 mm
- net RIGHT_MOTOR_DIR: track 0.00 -> 28.6 mm
- net LEFT_MOTOR_STEP: track 0.00 -> 28.3 mm
- net MPU_SDA: track 0.00 -> 27.9 mm, vias 0 -> 1
- net RIGHT_MOTOR_STEP: track 0.00 -> 27.0 mm
- net MPU_INTERRUPT: track 0.00 -> 23.1 mm, vias 0 -> 1
- net Net-(A1-Pad14): track 0.00 -> 21.1 mm
- net Net-(A2-Pad14): track 0.00 -> 21.1 mm
- net Net-(A2-Pad13): track 0.00 -> 17.5 mm
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Other:
- board size 66.7 x 59.7 mm -> 62.4 x 57.5 mm
- board text added: "BalanceBot by FrostieBot v0.4.5"
- board text removed: "BalanceBot by FrostieBot v0.3.4"
- board text removed: "VIN"
