File: design/balancebot.sch (KiCad schematic (older format))
At the start: 18 parts, among them J1 Power Header, J3 Passthrough, J4 Servo Interface, J5 Left Motor Interface, J6 Right Motor Interface, U1 ESP32, U2 TSR_1-2450, U3 GY-521

Commit message: update PCB design to revision 0.4.5
Parts:
- removed J1: Power Header, Connector_PinHeader_2.54mm:PinHeader_2x02_P2.54mm_Vertical, symbol Connector_Generic:Conn_02x02_Top_Bottom
- removed U2: TSR_1-2450, Converter_DCDC:Converter_DCDC_TRACO_TSR-1_THT, symbol Regulator_Switching:TSR_1-2450
- added U2: OKI-78SR-5/1.5-W36-C, Converter_DCDC:Converter_DCDC_muRata_OKI-78SR_Vertical, symbol Converter_DCDC:OKI-78SR-5_1.5-W36-C
- TB2: value 6.5V-36V -> 7V-36V
- U3: value GY-521 -> MPU6050
Connections:
- net +5V: now also U2.3 (OUT)
- net +VMOT: now also U2.1 (IN)
- net GND: now also U2.2 (GND)
- net MOTOR_ENABLE: now also J3.11 (Pin_11), U1.11 (IO25); no longer J3.9 (Pin_9), U1.9 (IO27)
- net RIGHT_MOTOR_DIR: now also J3.9 (Pin_9), U1.9 (IO27); no longer J3.10 (Pin_10), U1.10 (IO26)
- net RIGHT_MOTOR_STEP: now also J3.10 (Pin_10), U1.10 (IO26); no longer J3.11 (Pin_11), U1.11 (IO25)
Other:
- moved on the sheet: H1, H2, H3, H4, TB1, TB2
